Commit message: added in physics sim and a couple of other walking forms

File: kinematics/temp_quadruped.urdf (robot description, URDF)
Before this commit: robot quadruped, 13 links, 12 joints
Links:
- link BL_coxa: mass None -> 0.2; geometry collision cylinder length=0.05 radius=0.02; visual cylinder length=0.05 radius=0.02
- link BL_femur: mass None -> 0.2; geometry collision cylinder length=0.2 radius=0.02; visual cylinder length=0.2 radius=0.02
- link BL_tibia: mass None -> 0.2; geometry collision cylinder length=0.2 radius=0.015; collision sphere radius=0.02
- link BR_coxa: mass None -> 0.2; geometry collision cylinder length=0.05 radius=0.02; visual cylinder length=0.05 radius=0.02
- link BR_femur: mass None -> 0.2; geometry collision cylinder length=0.2 radius=0.02; visual cylinder length=0.2 radius=0.02
- link BR_tibia: mass None -> 0.2; geometry collision cylinder length=0.2 radius=0.015; collision sphere radius=0.02
- link FL_coxa: mass None -> 0.2; geometry collision cylinder length=0.05 radius=0.02; visual cylinder length=0.05 radius=0.02
- link FL_femur: mass None -> 0.2; geometry collision cylinder length=0.2 radius=0.02; visual cylinder length=0.2 radius=0.02
- link FL_tibia: mass None -> 0.2; geometry collision cylinder length=0.2 radius=0.015; collision sphere radius=0.02
- link FR_coxa: mass None -> 0.2; geometry collision cylinder length=0.05 radius=0.02; visual cylinder length=0.05 radius=0.02
- link FR_femur: mass None -> 0.2; geometry collision cylinder length=0.2 radius=0.02; visual cylinder length=0.2 radius=0.02
- link FR_tibia: mass None -> 0.2; geometry collision cylinder length=0.2 radius=0.015; collision sphere radius=0.02
- link base_link: mass None -> 2.0; geometry collision box size=0.4 0.2 0.05; visual box size=0.4 0.2 0.05
Joints:
- joint BL_knee_pitch: limit lower=-3.0 upper=3.0 effort=20 velocity=10 -> lower=-3.0 upper=3.0 effort=30 velocity=10
- joint BL_shoulder_pitch: limit lower=-1.5 upper=1.5 effort=20 velocity=10 -> lower=-1.5 upper=1.5 effort=30 velocity=10
- joint BL_shoulder_roll: limit lower=-1.5 upper=1.5 effort=20 velocity=10 -> lower=-1.5 upper=1.5 effort=30 velocity=10
- joint BR_knee_pitch: limit lower=-3.0 upper=3.0 effort=20 velocity=10 -> lower=-3.0 upper=3.0 effort=30 velocity=10
- joint BR_shoulder_pitch: limit lower=-1.5 upper=1.5 effort=20 velocity=10 -> lower=-1.5 upper=1.5 effort=30 velocity=10
- joint BR_shoulder_roll: limit lower=-1.5 upper=1.5 effort=20 velocity=10 -> lower=-1.5 upper=1.5 effort=30 velocity=10
- joint FL_knee_pitch: limit lower=-3.0 upper=3.0 effort=20 velocity=10 -> lower=-3.0 upper=3.0 effort=30 velocity=10
- joint FL_shoulder_pitch: limit lower=-1.5 upper=1.5 effort=20 velocity=10 -> lower=-1.5 upper=1.5 effort=30 velocity=10
- joint FL_shoulder_roll: limit lower=-1.5 upper=1.5 effort=20 velocity=10 -> lower=-1.5 upper=1.5 effort=30 velocity=10
- joint FR_knee_pitch: limit lower=-3.0 upper=3.0 effort=20 velocity=10 -> lower=-3.0 upper=3.0 effort=30 velocity=10
- joint FR_shoulder_pitch: limit lower=-1.5 upper=1.5 effort=20 velocity=10 -> lower=-1.5 upper=1.5 effort=30 velocity=10
- joint FR_shoulder_roll: limit lower=-1.5 upper=1.5 effort=20 velocity=10 -> lower=-1.5 upper=1.5 effort=30 velocity=10
